File: can-breakout.kicad_sch (KiCad schematic)
At the start: 0 parts

Commit message: feat: implemented breakout
Parts:
- added C1: 100nF, Capacitor_SMD:C_0402_1005Metric, symbol Device:C
- added C2: 4.7uF, Capacitor_SMD:C_0402_1005Metric, symbol Device:C
- added D1: SZNUP2105L, Package_TO_SOT_SMD:SOT-23, symbol Power_Protection:SZNUP2105L
- added J1: Conn_01x04, Connector_PinHeader_2.54mm:PinHeader_1x04_P2.54mm_Vertical, symbol Connector_Generic:Conn_01x04
- added J2: Conn_01x02, Connector_JST:JST_PH_B2B-PH-K_1x02_P2.00mm_Vertical, symbol Connector_Generic:Conn_01x02
- added R1: 120, Resistor_SMD:R_0402_1005Metric, symbol Device:R
- added R2, R3, R4: 10k, Resistor_SMD:R_0402_1005Metric, symbol Device:R
- added U1: SN65HVD230, Package_SO:SOIC-8_3.9x4.9mm_P1.27mm, symbol Interface_CAN_LIN:SN65HVD230
Connections:
- new net: R2.1, U1.8 (Rs)
- new net: R3.2, U1.1 (D)
- new net: R4.2, U1.4 (R)
- new net: D1.1 (K), J2.2 (Pin_2), R1.2, U1.6 (CANL)
- new net: D1.2 (K), J2.1 (Pin_1), R1.1, U1.7 (CANH)
- new net: J1.2 (Pin_2), R3.1
- new net: J1.3 (Pin_3), R4.1
- new net GND: C1.2, C2.2, D1.3 (A), J1.4 (Pin_4), R2.2, U1.2 (GND)
- new net VDD_3V3: C1.1, C2.1, J1.1 (Pin_1), U1.3 (VCC)
- no-connect marks 0 -> 1

Commit message: feat: completed board
Connections:
- net CANL: now reaches D1.1 (K), J2.2 (Pin_2), R1.2, U1.6 (CANL)
- net CANH: now reaches D1.2 (K), J2.1 (Pin_1), R1.1, U1.7 (CANH)
- net CAN_RX: now reaches J1.2 (Pin_2)
- net CAN_RX: now also R4.1; no longer R3.1
- net CAN_TX: now reaches J1.3 (Pin_3)
- net CAN_TX: now also R3.1; no longer R4.1
Changed lines of the file:
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@@
+	(wire
+		(pts
+			(xy 111.76 99.06) (xy 109.22 101.6)
+		)
+		(stroke
+			(width 0)
+			(type default)
+		)
+	)
+	(wire
+		(pts
+			(xy 104.14 99.06) (xy 109.22 99.06)
+		)
+		(stroke
+			(width 0)
+			(type default)
+		)
+	)
 	(wire
 		(pts
@@
 	(wire
 		(pts
+			(xy 123.19 99.06) (xy 111.76 99.06)
+		)
+		(stroke
+			(width 0)
+			(type default)
+		)
+	)
+	(wire
+		(pts
 			(xy 168.91 109.22) (xy 173.99 109.22)
 		)
@@
 	(wire
 		(pts
-			(xy 104.14 99.06) (xy 123.19 99.06)
+			(xy 111.76 101.6) (xy 123.19 101.6)
 		)
 		(stroke
@@
 	(wire
 		(pts
+			(xy 104.14 101.6) (xy 109.22 101.6)
+		)
+		(stroke
+			(width 0)
+			(type default)
+		)
+	)
+	(wire
+		(pts
 			(xy 130.81 99.06) (xy 140.97 99.06)
 		)
@@
 	(wire
 		(pts
+			(xy 109.22 99.06) (xy 111.76 101.6)
+		)
+		(stroke
+			(width 0)
+			(type default)
+		)
+	)
+	(wire
+		(pts
 			(xy 176.53 105.41) (xy 173.99 105.41)
 		)
@@
 	(wire
 		(pts
-			(xy 104.14 101.6) (xy 123.19 101.6)
-		)
-		(stroke
-			(width 0)
-			(type default)
-		)
-	)
-	(wire
-		(pts
 			(xy 130.81 101.6) (xy 140.97 101.6)
 		)
@@
 		)
 	)
+	(label "CAN_RX"
+		(at 115.57 101.6 0)
+		(effects
+			(font
+				(size 1.27 1.27)
+			)
+			(justify left bottom)
+		)
+	)
+	(label "CAN_TX"
+		(at 115.57 99.06 0)
+		(effects
+			(font
+				(size 1.27 1.27)
+			)
+			(justify left bottom)
+		)
+	)
+	(label "CANL"
+		(at 198.12 109.22 0)
+		(effects
+			(font
+				(size 1.27 1.27)
+			)
+			(justify left bottom)
+		)
+	)
+	(label "CANH"
+		(at 198.12 96.52 0)
+		(effects
+			(font
+				(size 1.27 1.27)
+			)
+			(justify left bottom)
+		)
+	)
